File: high-voltage-switch.kicad_pcb (KiCad board)
At the start: 2 copper layers, 79 x 74 mm, 35 parts, among them J1 Screw_Terminal_01x04, J2 Screw_Terminal_01x02, J3 Screw_Terminal_01x02, J4 Conn_02x04_Odd_Even, K1 G5Q-1A4-DC5, K2 G5Q-1A4-DC5, K3 G5Q-1A4-DC5, K4 G5Q-1A4-DC5, Q1 IRFZ34NPBF, Q2 IRFZ34NPBF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

Commit message: final version 1.0
Parts:
- HOLE_NW: renamed from REF**; value MountingHole_3.2mm_M3_DIN965 -> MountingHole_3.2mm_M3_DIN96
- renumbered REF** to HOLE_NE, REF** to HOLE_SE, REF** to HOLE_SW
Other:
- outline, holes or cut-outs redrawn
- board text added: "4 Channel 220 VAC Switch v1.0"
Changed lines of the file:
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@@
 			(outputformat 1)
 			(mirror no)
-			(drillshape 1)
+			(drillshape 0)
 			(scaleselection 1)
-			(outputdirectory "")
+			(outputdirectory "gerber-v1.0")
 		)
 	)
@@
 			)
 		)
-		(property "Datasheet" ""
+		(property "Datasheet" "~"
 			(at 0 0 0)
 			(layer "F.Fab")
@@
 			)
 		)
-		(property "Datasheet" ""
+		(property "Datasheet" "~"
 			(at 0 0 90)
 			(layer "F.Fab")
@@
 			)
 		)
-		(property "Datasheet" ""
+		(property "Datasheet" "~"
 			(at 0 0 0)
 			(layer "F.Fab")
@@
 			)
 		)
-		(property "Datasheet" ""
+		(property "Datasheet" "~"
 			(at 0 0 0)
 			(layer "F.Fab")
@@
 			)
 		)
-		(property "Datasheet" ""
+		(property "Datasheet" "~"
 			(at 0 0 90)
 			(layer "F.Fab")
@@
 			)
 		)
-		(property "Datasheet" ""
+		(property "Datasheet" "~"
 			(at 0 0 0)
 			(layer "F.Fab")
@@
 			)
 		)
-		(property "Datasheet" ""
+		(property "Datasheet" "~"
 			(at 0 0 90)
 			(layer "F.Fab")
@@
 			)
 		)
-		(property "Datasheet" ""
+		(property "Datasheet" "~"
 			(at 0 0 0)
 			(layer "F.Fab")
@@
 			)
 		)
-		(property "Datasheet" ""
+		(property "Datasheet" "~"
 			(at 0 0 0)
 			(layer "F.Fab")
@@
 			)
 		)
-		(property "Datasheet" ""
+		(property "Datasheet" "~"
 			(at 0 0 270)
 			(unlocked yes)
@@
 			)
 		)
-		(property "Datasheet" ""
+		(property "Datasheet" "~"
 			(at 0 0 0)
 			(layer "F.Fab")
@@
 		(descr "Mounting Hole 3.2mm, M3, no annular, generated by kicad-footprint-generator mountinghole.py")
 		(tags "mountinghole M3 DIN965")
-		(property "Reference" "REF**"
+		(property "Reference" "HOLE_NW"
 			(at 0 -3.75 0)
 			(layer "F.SilkS")
@@
 			)
 		)
-		(property "Value" "MountingHole_3.2mm_M3_DIN965"
+		(property "Value" "MountingHole_3.2mm_M3_DIN96"
 			(at 0 3.75 0)
 			(layer "F.Fab")
@@
 			)
 		)
-		(property "Datasheet" ""
+		(property "Datasheet" "~"
 			(at 0 0 90)
 			(unlocked yes)
@@
 			)
 		)
-		(property "Datasheet" ""
+		(property "Datasheet" "~"
 			(at 0 0 0)
 			(layer "F.Fab")
@@
 		(sheetfile "high-voltage-switch.kicad_sch")
 		(attr through_hole)
+		(fp_rect
+			(start -2 -6.5)
+			(end 27.5 46.5)
+			(stroke
+				(width 0.05)
+				(type default)
+			)
+			(fill no)
+			(layer "B.CrtYd")
+		)
 		(fp_line
 			(start 9.525 45.56)
@@
 			(layer "F.Fab")
 		)
-		(pad "" thru_hole circle
+		(pad "" np_thru_hole circle
 			(at 0.73 -4 270)
 			(size 3 3)
 			(drill 3)
 			(layers "*.Cu" "*.Mask")
-			(remove_unused_layers no)
 		)
-		(pad "" thru_hole circle
+		(pad "" np_thru_hole circle
 			(at 0.73 43.56 270)
 			(size 3 3)
 			(drill 3)
 			(layers "*.Cu" "*.Mask")
-			(remove_unused_layers no)
 		)
-		(pad "" thru_hole circle
+		(pad "" np_thru_hole circle
 			(at 24.67 -4 270)
 			(size 3 3)
 			(drill 3)
 			(layers "*.Cu" "*.Mask")
-			(remove_unused_layers no)
 		)
-		(pad "" thru_hole circle
+		(pad "" np_thru_hole circle
 			(at 24.67 43.56 270)
 			(size 3 3)
 			(drill 3)
 			(layers "*.Cu" "*.Mask")
-			(remove_unused_layers no)
 		)
 		(pad "1" thru_hole circle
@@
 			(net 24 "unconnected-(U1-EN-Pad1)")
 			(pinfunction "EN")
-			(pintype "input")
+			(pintype "input+no_connect")
 		)
 		(pad "2" thru_hole circle
@@
 			(net 36 "unconnected-(U1-VP-Pad2)")
 			(pinfunction "VP")
-			(pintype "input")
+			(pintype "input+no_connect")
 		)
 		(pad "3" thru_hole circle
@@
 			(net 32 "unconnected-(U1-VN-Pad3)")
 			(pinfunction "VN")
-			(pintype "input")
+			(pintype "input+no_connect")
 		)
 		(pad "4" thru_hole circle
@@
 			(net 28 "unconnected-(U1-D25-Pad8)")
 			(pinfunction "D25")
-			(pintype "bidirectional")
+			(pintype "bidirectional+no_connect")
 		)
 		(pad "9" thru_hole circle
@@
 			(net 31 "unconnected-(U1-D26-Pad9)")
 			(pinfunction "D26")
-			(pintype "bidirectional")
+			(pintype "bidirectional+no_connect")
 		)
 		(pad "10" thru_hole circle
@@
 			(net 27 "unconnected-(U1-D27-Pad10)")
 			(pinfunction "D27")
-			(pintype "bidirectional")
+			(pintype "bidirectional+no_connect")
 		)
 		(pad "11" thru_hole circle
@@
 			(net 25 "unconnected-(U1-D14-Pad11)")
 			(pinfunction "D14")
-			(pintype "bidirectional")
+			(pintype "bidirectional+no_connect")
 		)
 		(pad "12" thru_hole circle
@@
 			(net 33 "unconnected-(U1-D12-Pad12)")
 			(pinfunction "D12")
-			(pintype "bidirectional")
+			(pintype "bidirectional+no_connect")
 		)
 		(pad "13" thru_hole circle
@@
 			(net 16 "unconnected-(U1-D13-Pad13)")
 			(pinfunction "D13")
-			(pintype "bidirectional")
+			(pintype "bidirectional+no_connect")
 		)
 		(pad "14" thru_hole circle
@@
 			(net 19 "unconnected-(U1-D23-Pad16)")
 			(pinfunction "D23")
-			(pintype "bidirectional")
+			(pintype "bidirectional+no_connect")
 		)
 		(pad "17" thru_hole circle
@@
 			(net 34 "unconnected-(U1-D22-Pad17)")
 			(pinfunction "D22")
-			(pintype "bidirectional")
+			(pintype "bidirectional+no_connect")
 		)
 		(pad "18" thru_hole circle
@@
 			(net 18 "unconnected-(U1-D21-Pad20)")
 			(pinfunction "D21")
-			(pintype "bidirectional")
+			(pintype "bidirectional+no_connect")
 		)
 		(pad "21" thru_hole circle
@@
 			(net 20 "unconnected-(U1-D19-Pad21)")
 			(pinfunction "D19")
-			(pintype "bidirectional")
+			(pintype "bidirectional+no_connect")
 		)
 		(pad "22" thru_hole circle
@@
 			(net 39 "unconnected-(U1-D18-Pad22)")
 			(pinfunction "D18")
-			(pintype "bidirectional")
+			(pintype "bidirectional+no_connect")
 		)
 		(pad "23" thru_hole circle
@@
 			(net 42 "unconnected-(U1-TX2-Pad24)")
 			(pinfunction "TX2")
-			(pintype "bidirectional")
+			(pintype "bidirectional+no_connect")
 		)
 		(pad "25" thru_hole circle
@@
 			(net 40 "unconnected-(U1-RX2-Pad25)")
 			(pinfunction "RX2")
-			(pintype "bidirectional")
+			(pintype "bidirectional+no_connect")
 		)
 		(pad "26" thru_hole circle
@@
 			(net 41 "unconnected-(U1-D4-Pad26)")
 			(pinfunction "D4")
-			(pintype "bidirectional")
+			(pintype "bidirectional+no_connect")
 		)
 		(pad "27" thru_hole circle
@@
 			(net 23 "unconnected-(U1-D2-Pad27)")
 			(pinfunction "D2")
-			(pintype "bidirectional")
+			(pintype "bidirectional+no_connect")
 		)
 		(pad "28" thru_hole circle
@@
 			(net 38 "unconnected-(U1-3V3-Pad30)")
 			(pinfunction "3V3")
-			(pintype "power_out")
+			(pintype "power_out+no_connect")
 		)
 		(embedded_fonts no)
@@
 			)
 		)
-		(property "Datasheet" ""
+		(property "Datasheet" "~"
 			(at 0 0 0)
 			(layer "F.Fab")
@@
 			)
 		)
-		(property "Datasheet" ""
+		(property "Datasheet" "~"
 			(at 0 0 90)
 			(layer "F.Fab")
@@
 			)
 		)
-		(property "Datasheet" ""
+		(property "Datasheet" "~"
 			(at 0 0 90)
 			(layer "F.Fab")
@@
 		(descr "Mounting Hole 3.2mm, M3, no annular, generated by kicad-footprint-generator mountinghole.py")
 		(tags "mountinghole M3 DIN965")
-		(property "Reference" "REF**"
+		(property "Reference" "HOLE_SE"
 			(at 0 -3.75 0)
 			(layer "F.SilkS")
@@
 			)
 		)
-		(property "Datasheet" ""
+		(property "Datasheet" "~"
 			(at 0 0 90)
 			(layer "F.Fab")
@@
 		(descr "Mounting Hole 3.2mm, M3, no annular, generated by kicad-footprint-generator mountinghole.py")
 		(tags "mountinghole M3 DIN965")
-		(property "Reference" "REF**"
+		(property "Reference" "HOLE_NE"
 			(at 0 -3.75 0)
 			(layer "F.SilkS")
@@
 			)
 		)
-		(property "Datasheet" ""
+		(property "Datasheet" "~"
 			(at 0 0 0)
 			(layer "F.Fab")
@@
 			)
 		)
-		(property "Datasheet" ""
+		(property "Datasheet" "~"
 			(at 0 0 0)
 			(layer "F.Fab")
@@
 			)
 		)
-		(property "Datasheet" ""
+		(property "Datasheet" "~"
 			(at 0 0 0)
 			(layer "F.Fab")
@@
 			)
 		)
-		(property "Datasheet" ""
+		(property "Datasheet" "~"
 			(at 0 0 0)
 			(layer "F.Fab")
@@
 			)
 		)
-		(property "Datasheet" ""
+		(property "Datasheet" "~"
 			(at 0 0 0)
 			(layer "F.Fab")
@@
 		(descr "Mounting Hole 3.2mm, M3, no annular, generated by kicad-footprint-generator mountinghole.py")
 		(tags "mountinghole M3 DIN965")
-		(property "Reference" "REF**"
+		(property "Reference" "HOLE_SW"
 			(at 0 -3.75 0)
 			(layer "F.SilkS")
@@
 		(embedded_fonts no)
 	)
+	(gr_arc
+		(start 124 50)
+		(mid 127.535534 51.464466)
+		(end 129 55)
+		(stroke
+			(width 0.05)
+			(type default)
+		)
+		(layer "Edge.Cuts")
+	)
 	(gr_line
-		(start 50 50)
-		(end 50 124)
+		(start 55 50)
+		(end 124 50)
+		(stroke
+			(width 0.05)
+			(type default)
+		)
+		(layer "Edge.Cuts")
+	)
+	(gr_arc
+		(start 50 55)
+		(mid 51.464466 51.464466)
+		(end 55 50)
 		(stroke
 			(width 0.05)
@@
 	)
 	(gr_line
-		(start 50 124)
-		(end 129 124)
+		(start 50 119)
+		(end 50 55)
 		(stroke
 			(width 0.05)
@@
 	)
 	(gr_line
-		(start 129 124)
-		(end 129 50)
+		(start 129 55)
+		(end 129 119)
+		(stroke
+			(width 0.05)
+			(type default)
+		)
+		(layer "Edge.Cuts")
+	)
+	(gr_arc
+		(start 55 124)
+		(mid 51.464466 122.535534)
+		(end 50 119)
+		(stroke
+			(width 0.05)
+			(type default)
+		)
+		(layer "Edge.Cuts")
+	)
+	(gr_arc
+		(start 129 119)
+		(mid 127.535534 122.535534)
+		(end 124 124)
 		(stroke
 			(width 0.05)
@@
 	)
 	(gr_line
-		(start 50 50)
-		(end 129 50)
+		(start 124 124)
+		(end 55 124)
 		(stroke
 			(width 0.05)
@@
 			)
 			(justify left bottom)
+		)
+	)
+	(gr_text "4 Channel 220 VAC Switch v1.0"
+		(at 60.4 123.3 0)
+		(layer "F.SilkS")
+		(effects
+			(font
+				(size 1.5 1.5)
+				(thickness 0.2)
+			)
+			(justify left bottom)
