File: high-voltage-switch.kicad_sch (KiCad schematic)
At the start: 31 parts, among them J1 Screw_Terminal_01x04, J2 Screw_Terminal_01x02, J3 Screw_Terminal_01x02, J4 Conn_02x04_Odd_Even, K1 G5Q-1A4-DC5, K2 G5Q-1A4-DC5, K3 G5Q-1A4-DC5, K4 G5Q-1A4-DC5, Q1 IRFZ34NPBF, Q2 IRFZ34NPBF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

Commit message: final version 1.0
Connections:
- no-connect marks 0 -> 19
Changed lines of the file:
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@@
+	)
+	(junction
+		(at 21.59 35.56)
+		(diameter 0)
+		(color 0 0 0 0)
 	)
 	(junction
@@
 		(color 0 0 0 0)
 	)
+	(no_connect
+		(at 68.58 88.9)
+	)
+	(no_connect
+		(at 68.58 63.5)
+	)
+	(no_connect
+		(at 68.58 81.28)
+	)
+	(no_connect
+		(at 68.58 86.36)
+	)
+	(no_connect
+		(at 99.06 81.28)
+	)
+	(no_connect
+		(at 99.06 58.42)
+	)
+	(no_connect
+		(at 68.58 83.82)
+	)
+	(no_connect
+		(at 68.58 58.42)
+	)
+	(no_connect
+		(at 68.58 76.2)
+	)
+	(no_connect
+		(at 68.58 60.96)
+	)
+	(no_connect
+		(at 99.06 86.36)
+	)
+	(no_connect
+		(at 99.06 71.12)
+	)
+	(no_connect
+		(at 68.58 78.74)
+	)
+	(no_connect
+		(at 99.06 60.96)
+	)
+	(no_connect
+		(at 99.06 93.98)
+	)
+	(no_connect
+		(at 99.06 73.66)
+	)
+	(no_connect
+		(at 99.06 68.58)
+	)
+	(no_connect
+		(at 99.06 83.82)
+	)
+	(no_connect
+		(at 99.06 78.74)
+	)
 	(wire
 		(pts
@@
 	(wire
 		(pts
+			(xy 17.78 35.56) (xy 21.59 35.56)
+		)
+		(stroke
+			(width 0)
+			(type default)
+		)
+	)
+	(wire
+		(pts
 			(xy 40.64 49.53) (xy 33.02 49.53)
 		)
@@
 		(pts
 			(xy 40.64 66.04) (xy 33.02 66.04)
+		)
+		(stroke
+			(width 0)
+			(type default)
+		)
+	)
+	(wire
+		(pts
+			(xy 17.78 26.67) (xy 17.78 35.56)
 		)
 		(stroke
@@
 					(unit 1)
 				)
+			)
+		)
+	)
+	(symbol
+		(lib_id "power:PWR_FLAG")
+		(at 17.78 26.67 0)
+		(unit 1)
+		(exclude_from_sim no)
+		(in_bom yes)
+		(on_board yes)
+		(dnp no)
+		(fields_autoplaced yes)
+		(property "Reference" "#FLG01"
+			(at 17.78 24.765 0)
+			(effects
+				(font
+					(size 1.27 1.27)
+				)
+				(hide yes)
+			)
+		)
+		(property "Value" "PWR_FLAG"
+			(at 17.78 22.5369 0)
+			(effects
+				(font
+					(size 1.27 1.27)
+				)
+			)
+		)
+		(property "Footprint" ""
+			(at 17.78 26.67 0)
+			(effects
+				(font
+					(size 1.27 1.27)
+				)
+				(hide yes)
+			)
+		)
+		(property "Datasheet" "~"
+			(at 17.78 26.67 0)
+			(effects
+				(font
+					(size 1.27 1.27)
+				)
+				(hide yes)
+			)
+		)
+		(property "Description" "Special symbol for telling ERC where power comes from"
+			(at 17.78 26.67 0)
+			(effects
+				(font
+					(size 1.27 1.27)
+				)
+				(hide yes)
+			)
+		)
+		(pin "1"
+		)
+		(instances
+			(project ""
+				(path "/8ed25bdd-aede-4325-9d77-6e039a30837a"
+					(reference "#FLG01")
+					(unit 1)
+				)
